Commit message: feat: improve readme about /low_state msg source

File: booster_dataset/utils/T1_7DofArm_Serial.urdf (robot description, URDF)
Before this commit: robot T1, 30 links, 29 joints
Links:
- link AL3: geometry visual mesh filename=meshes/AL3.STL
- link AL4: mass 0.2984 -> 0.5570; geometry visual mesh filename=meshes/AL4.STL
- link AL5: mass 0.42219 -> 0.43402
- link AL6: mass 0.26532 -> 0.47922
- link AR3: geometry visual mesh filename=meshes/AR3.STL
- link AR4: mass 0.3599 -> 0.5570; geometry visual mesh filename=meshes/AR4.STL
- link AR6: mass 0.28215 -> 0.47922
- link left_hand_link: mass 0.24875 -> 0.30603; geometry visual mesh filename=meshes/AL7.STL
- link right_hand_link: mass 0.24612 -> 0.30603; geometry visual mesh filename=meshes/AR7.STL
Joints:
- removed joint Waist
- added joint Waist_Joint: type revolute, parent Trunk, child Waist, origin xyz=0.0625 0 -0.1155 rpy=0 0 0, axis 0 0 1, limit lower=-1.57 upper=1.57 effort=30 velocity=10.88
- joint Left_Elbow_Pitch: limit lower=-2.27 upper=2.27 effort=18 velocity=18.84 -> lower=-2.234 upper=2.234 effort=18 velocity=18.84
- joint Left_Elbow_Yaw: limit lower=-2.27 upper=2.27 effort=18 velocity=18.84 -> lower=-2.1402 upper=1.6844 effort=18 velocity=18.84
- joint Left_Hand_Roll: limit lower=-2.27 upper=2.27 effort=18 velocity=18.84 -> lower=-0.758 upper=1.4285 effort=7 velocity=12.56
- joint Left_Shoulder_Pitch: limit lower=-3.31 upper=1.22 effort=18 velocity=18.84 -> lower=-3.29 upper=1.18 effort=18 velocity=18.84
- joint Left_Shoulder_Roll: limit lower=-1.74 upper=1.57 effort=18 velocity=18.84 -> lower=-1.577 upper=1.7055 effort=18 velocity=18.84
- joint Left_Wrist_Pitch: limit lower=-2.27 upper=2.27 effort=18 velocity=18.84 -> lower=-2.5821 upper=2.5821 effort=7 velocity=12.56
- joint Left_Wrist_Yaw: limit lower=-2.27 upper=2.27 effort=18 velocity=18.84 -> lower=-1.8185 upper=1.4261 effort=18 velocity=18.84
- joint Right_Elbow_Pitch: limit lower=-2.27 upper=2.27 effort=18 velocity=18.84 -> lower=-2.234 upper=2.234 effort=18 velocity=18.84
- joint Right_Elbow_Yaw: limit lower=-2.27 upper=2.27 effort=18 velocity=18.84 -> lower=-1.6844 upper=2.1402 effort=18 velocity=18.84
- joint Right_Hand_Roll: limit lower=-2.27 upper=2.27 effort=18 velocity=18.84 -> lower=-1.4285 upper=0.758 effort=7 velocity=12.56
- joint Right_Shoulder_Pitch: limit lower=-3.31 upper=1.22 effort=18 velocity=18.84 -> lower=-3.29 upper=1.1868 effort=18 velocity=18.84
- joint Right_Shoulder_Roll: limit lower=-1.57 upper=1.74 effort=18 velocity=18.84 -> lower=-1.7055 upper=1.577 effort=18 velocity=18.84
- joint Right_Wrist_Pitch: limit lower=-2.27 upper=2.27 effort=18 velocity=18.84 -> lower=-2.5821 upper=2.5821 effort=7 velocity=12.56
- joint Right_Wrist_Yaw: limit lower=-2.27 upper=2.27 effort=18 velocity=18.84 -> lower=-1.4261 upper=1.8185 effort=18 velocity=18.84
